File: KiCad_Traffic_Light_Controller/KiCad_Traffic_Light_Controller.kicad_pcb (KiCad board)
At the start: 2 copper layers, 64 parts, among them J1 Conn_02x08_Odd_Even, J2 Conn_02x08_Odd_Even, J3 Conn_02x05_Odd_Even, J4 +5V, SW1 RST, SW2 OVR, SW3 EN, U1 SM420561N, U2 SM420561N, U3 LM1117DT-3.3

Commit message: CONNECTIONS 1
Parts:
- moved D4 2.54 mm to (122.5, 104.0), turned to 180 degrees
- moved D5 2.54 mm to (122.5, 114.5), turned to 180 degrees
- moved R23 2.45 mm to (207.5, 61.5)
- moved R24 2.45 mm to (207.5, 73.0)
- moved R1 2.40 mm to (188.0, 54.0)
- moved R2 2.40 mm to (192.0, 54.0)
- moved R6 2.40 mm to (184.0, 54.0)
- moved R7 2.40 mm to (180.0, 54.0)
- moved D6 2.27 mm to (122.5, 124.5), turned to 180 degrees
- moved R3 1.50 mm to (187.5, 81.5)
- moved R4 1.50 mm to (184.0, 81.5)
- moved R5 1.50 mm to (180.5, 81.5)
- moved R8 1.50 mm to (191.0, 81.5)
- turned R31 to 0 degrees
Routing:
- net GND: track 0.00 -> 278.3 mm, vias 0 -> 3
- net /+5V: track 0.00 -> 98.9 mm
- net /+3.3V: track 0.00 -> 85.9 mm
- net Net-(D13-A): track 0.00 -> 13.5 mm
- net Net-(D12-A): track 0.00 -> 12.7 mm
- net /OVR: track 0.00 -> 8.10 mm
- net Net-(D9-K): track 0.00 -> 7.91 mm
- net Net-(D11-A): track 0.00 -> 6.68 mm
- net Net-(D6-K): track 0.00 -> 6.50 mm
- net Net-(U1-F): track 0.00 -> 5.33 mm
- net Net-(U1-A): track 0.00 -> 5.31 mm
- net Net-(U1-C): track 0.00 -> 5.26 mm
- net Net-(U2-G): track 0.00 -> 5.14 mm
- net Net-(U2-B): track 0.00 -> 5.14 mm
- net Net-(U1-D): track 0.00 -> 5.05 mm
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
Commit message: NEW UPD
Parts:
- C2, C3, C5: value 0.22u -> 0.22μ
- D1: value GREEN -> NSC_GRN
- D10: value RED -> EWP_RED
- D2: value YELLOW -> NSC_YLW
- D3: value RED -> NSC_RED
- D4: value GREEN -> EWC_GRN
- D5: value YELLOW -> EWC_YLW
- D6: value RED -> EWC_RED
- D7: value GREEN -> NSP_GRN
- D8: value RED -> NSP_RED
- D9: value GREEN -> EWP_GRN
- moved H3 291.7 mm to (219.0, 39.5)
- moved H4 283.5 mm to (219.0, 135.0)
- moved H1 153.1 mm to (77.5, 40.0)
- moved H2 144.6 mm to (77.5, 135.0)
Connections:
- D10 pad 2: /NSC_RED -> /EWP_RED
- D7 pad 2: /NSC_GRN -> /NSP_GRN
- D8 pad 2: /NSC_RED -> /NSP_RED
- D9 pad 2: /NSC_GRN -> /EWP_GRN
- J1 pad 1: /+3.3 -> /+3.3V
- J2 pad 1: /+3.3 -> /+3.3V
Routing:
- net GND: track 278.3 -> 505.7 mm, vias 3 -> 4
- net /+3.3V: track 85.9 -> 311.8 mm, vias 0 -> 4
- net /EN: track 0.00 -> 180.7 mm
- net /RST: track 0.00 -> 164.8 mm, vias 0 -> 2
- net /OVR: track 8.10 -> 160.7 mm, vias 0 -> 2
- net /NS_HEX_A: track 0.00 -> 122.9 mm
- net /NS_HEX_B: track 0.00 -> 108.7 mm
- net /NSP_RED: track 0.00 -> 88.1 mm
- net /EW_HEX_D: track 0.00 -> 88.1 mm
- net /NSC_GRN: track 0.00 -> 86.8 mm, vias 0 -> 2
- net /NSP_GRN: track 0.00 -> 83.9 mm
- net /EW_HEX_C: track 0.00 -> 80.9 mm
- net /NS_HEX_F: track 0.00 -> 75.6 mm
- net /EW_HEX_E: track 0.00 -> 73.6 mm, vias 0 -> 1
- net /EW_HEX_DP: track 0.00 -> 72.8 mm, vias 0 -> 1
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Other:
- board text added: "+3V3"
- board text added: "+5V"
- board text added: "A"
- board text added: "B"
- board text added: "C"
- board text added: "CAR"
- board text added: "Control Logic Connector"
- board text added: "D"
- board text added: "DP"
- board text added: "E"
- board text added: "E-W"
- board text added: "EAST-WEST TRAFFIC LIGHTS"
- board text added: "EN"
- board text added: "ENABLE"
- board text added: "EW Connector"
- board text added: "F"
- board text added: "G"
- board text added: "GND"
- board text added: "GND GND"
- board text added: "It manages traffic flow for two perpendicular roads:"
- board text added: "N-S"
- board text added: "NORTH-SOUTH TRAFFIC LIGHTS"
- board text added: "NS Connector"
- board text added: "North-South (NS) and East-West (EW)."
- board text added: "OVERRIDE"
- board text added: "OVR"
- board text added: "PED"
- board text added: "R"
- board text added: "RESET"
- board text added: "RHILE L. GALPO 22 April 2026 Computer Engineering Technology Department Technological University of the Philippines Visayas"
- board text added: "RST"
- board text added: "Traffic Light Controller board for Finite State Machine (FSM) Demo."
- board text added: "Y"
